File: hardware/bpw34_opa381_frontend/bpw34_opa381_frontend.kicad_sch (KiCad schematic)
At the start: 0 parts

Commit message: Add v0.1-A power and reference schematic
Parts:
- added C1, C3, C5: 4.7uF, Capacitor_SMD:C_0603_1608Metric, symbol Device:C
- added C2, C4, C6, C7: 100nF, Capacitor_SMD:C_0603_1608Metric, symbol Device:C
- added C8, C9: 1uF, Capacitor_SMD:C_0603_1608Metric, symbol Device:C
- added FB1: BLM18AG601SN1D, Inductor_SMD:L_0603_1608Metric, symbol Device:FerriteBead
- added J1: Conn_01x03, symbol Connector_Generic:Conn_01x03
- added R1: 10k, Resistor_SMD:R_0603_1608Metric, symbol Device:R
- added U1: LP5907MFX-3.3/NOPB, Package_TO_SOT_SMD:SOT-23-5, symbol Regulator_Linear:LP5907MFX-3.3
- added U2: REF3312AIDBZR, Package_TO_SOT_SMD:SOT-23, symbol FrontEnd_Custom:REF3312AIDBZR
Connections:
- new net +5V_FILTER: C3.1, C4.1, FB1.2, U1.1 (IN), U1.3 (EN)
- new net +5V_IN: C1.1, C2.1, FB1.1, J1.1 (Pin_1)
- new net ADC_OUT: J1.3 (Pin_3)
- new net AGND: C1.2, C2.2, C3.2, C4.2, C5.2, C6.2, C7.2, C8.2, C9.2, J1.2 (Pin_2), U1.2 (GND), U2.3 (GND)
- new net AVDD_3V3: C5.1, C6.1, C7.1, U1.5 (OUT), U2.1 (IN)
- new net VBIAS_1V25: C9.1, R1.2
- new net VREF_RAW: C8.1, R1.1, U2.2 (OUT)
- no-connect marks 0 -> 1

Commit message: Add v0.1-B TIA and ADC filter schematic
Parts:
- added C10: 100nF, Capacitor_SMD:C_0603_1608Metric, symbol Device:C
- added C11: 1uF, Capacitor_SMD:C_0603_1608Metric, symbol Device:C
- added C12: 33nF, Capacitor_SMD:C_0603_1608Metric, symbol Device:C
- added CF1: 15pF, Capacitor_SMD:C_0603_1608Metric, symbol Device:C
- added D1: BPW34, FrontEnd_Footprints:BPW34_Vishay_P5.10mm, symbol FrontEnd_Custom:BPW34_Vishay
- added R2: 1k, Resistor_SMD:R_1206_3216Metric, symbol Device:R
- added RF1: 1M, Resistor_SMD:R_1206_3216Metric, symbol Device:R
- added U3: OPA381AIDGKR, Package_SO:VSSOP-8_3x3mm_P0.65mm, symbol FrontEnd_Custom:OPA381AIDGKR
Connections:
- net ADC_OUT: now also C12.2, R2.2
- net AGND: now also C10.1, C11.1, C12.1, D1.1 (A), U3.4 (V-)
- net AVDD_3V3: now also C10.2, C11.2, U3.7 (V+)
- net VBIAS_1V25: now also U3.3 (+IN)
- new net SUM: CF1.1, D1.2 (K), RF1.1, U3.2 (-IN)
- new net TIA_OUT: CF1.2, R2.1, RF1.2, U3.6 (OUT)
- no-connect marks 1 -> 4

Commit message: Complete v0.1 schematic with calibration and test points
Parts:
- added J2: Conn_01x02, symbol Connector_Generic:Conn_01x02
- added R3: 100M, Resistor_SMD:R_1206_3216Metric, symbol Device:R
- added SJ1: OPEN, Jumper:SolderJumper-2_P1.3mm_Open_RoundedPad1.0x1.5mm, symbol Jumper:SolderJumper_2_Open
- added TP1: +5V_IN, TestPoint:TestPoint_Pad_D1.0mm, symbol Connector:TestPoint
- added TP10: CAL_IN, TestPoint:TestPoint_Pad_D1.0mm, symbol Connector:TestPoint
- added TP2: +5V_FILTER, TestPoint:TestPoint_Pad_D1.0mm, symbol Connector:TestPoint
- added TP3: AVDD_3V3, TestPoint:TestPoint_Pad_D1.0mm, symbol Connector:TestPoint
- added TP4: VREF_RAW, TestPoint:TestPoint_Pad_D1.0mm, symbol Connector:TestPoint
- added TP5: VBIAS_1V25, TestPoint:TestPoint_Pad_D1.0mm, symbol Connector:TestPoint
- added TP6: SUM_HIZ, FrontEnd_Footprints:TestPoint_Pad_D0.8mm, symbol Connector:TestPoint
- added TP7: TIA_OUT, FrontEnd_Footprints:TestPoint_Pad_D1.2mm, symbol Connector:TestPoint
- added TP8: ADC_OUT, FrontEnd_Footprints:TestPoint_Pad_D1.2mm, symbol Connector:TestPoint
- added TP9: AGND, FrontEnd_Footprints:TestPoint_Pad_D1.2mm, symbol Connector:TestPoint
Connections:
- net +5V_FILTER: now also TP2.1
- net +5V_IN: now also TP1.1
- net ADC_OUT: now also TP8.1
- net AGND: now also J2.2 (Pin_2), TP9.1
- net AVDD_3V3: now also TP3.1
- net SUM: now also SJ1.2 (B), TP6.1
- net TIA_OUT: now also TP7.1
- net VBIAS_1V25: now also TP5.1
- net VREF_RAW: now also TP4.1
- new net CAL_IN: J2.1 (Pin_1), R3.1, TP10.1
- new net CAL_R_NODE: R3.2, SJ1.1 (A)
Other:
- note added: "CALIBRATION"
- note added: "TEST POINTS"

Commit message: Freeze J1 and J2 production connectors
Parts:
- J1: footprint (none) -> Connector_JST:JST_PH_S3B-PH-SM4-TB_1x03-1MP_P2.00mm_Horizontal; LCSC (none) -> C265101; MPN (none) -> S3B-PH-SM4-TB(LF)(SN); Manufacturer (none) -> JST
- J2: footprint (none) -> Connector_JST:JST_PH_S2B-PH-SM4-TB_1x02-1MP_P2.00mm_Horizontal; LCSC (none) -> C295747; MPN (none) -> S2B-PH-SM4-TB(LF)(SN); Manufacturer (none) -> JST
Changed lines of the file:
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@@
 				(font
 (size 1.27 1.27))))
-		(property "Footprint" ""
+		(property "Footprint" "Connector_JST:JST_PH_S3B-PH-SM4-TB_1x03-1MP_P2.00mm_Horizontal"
 (at 38.10 50.80 0)
 			(effects
@@
 (hide yes)))
 		(property "Description" ""
+(at 38.10 50.80 0)
+			(effects
+				(font
+(size 1.27 1.27))
+(hide yes)))
+		(property "Manufacturer" "JST"
+(at 38.10 50.80 0)
+			(effects
+				(font
+(size 1.27 1.27))
+(hide yes)))
+		(property "MPN" "S3B-PH-SM4-TB(LF)(SN)"
+(at 38.10 50.80 0)
+			(effects
+				(font
+(size 1.27 1.27))
+(hide yes)))
+		(property "LCSC" "C265101"
 (at 38.10 50.80 0)
 			(effects
@@
 			(at 34.29 119.38 0)
 			(effects (font (size 1.27 1.27)) ))
-		(property "Footprint" ""
+		(property "Footprint" "Connector_JST:JST_PH_S2B-PH-SM4-TB_1x02-1MP_P2.00mm_Horizontal"
 			(at 35.56 124.46 0)
 			(effects (font (size 1.27 1.27)) (hide yes) ))
@@
 			(at 35.56 124.46 0)
 			(effects (font (size 1.27 1.27)) (hide yes) ))
+		(property "Manufacturer" "JST"
+			(at 35.56 124.46 0)
+			(effects (font (size 1.27 1.27)) (hide yes) ))
+		(property "MPN" "S2B-PH-SM4-TB(LF)(SN)"
+			(at 35.56 124.46 0)
+			(effects (font (size 1.27 1.27)) (hide yes) ))
+		(property "LCSC" "C295747"
+			(at 35.56 124.46 0)
+			(effects (font (size 1.27 1.27)) (hide yes) ))
