File: hardware/bpw34_opa381_frontend/bpw34_opa381_frontend.kicad_pcb (KiCad board)
At the start: 2 copper layers, 45 x 30 mm, 35 parts, among them J1 Conn_01x03, J2 Conn_01x02, U1 LP5907MFX-3.3/NOPB, U2 REF3312AIDBZR, U3 OPA381AIDGKR

Commit message: Complete v0.3 critical analog routing
Routing:
- net SUM: track 0.00 -> 16.5 mm
- net TIA_OUT: track 0.00 -> 15.8 mm
- net AVDD_3V3: track 0.00 -> 2.35 mm
- net AGND: track 0.00 -> 1.23 mm, vias 0 -> 2
Changed lines of the file:
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@@
 		(layer "Edge.Cuts")
+	)
+	(segment
+		(start 116.8 109.475)
+		(end 117.4 109.475)
+		(width 0.25)
+		(layer "F.Cu")
+		(net "AGND")
+	)
+	(segment
+		(start 110.5375 109.975)
+		(end 110.5375 110.6)
+		(width 0.25)
+		(layer "F.Cu")
+		(net "AGND")
+	)
+	(via
+		(at 117.4 109.475)
+		(size 0.6)
+		(drill 0.3)
+		(layers "F.Cu" "B.Cu")
+		(net "AGND")
+	)
+	(via
+		(at 110.5375 110.6)
+		(size 0.6)
+		(drill 0.3)
+		(layers "F.Cu" "B.Cu")
+		(net "AGND")
+	)
+	(segment
+		(start 111.75 111.525)
+		(end 111.875 112)
+		(width 0.2)
+		(layer "F.Cu")
+		(net "SUM")
+	)
+	(segment
+		(start 106.65 111.55)
+		(end 106.15 112.05)
+		(width 0.2)
+		(layer "F.Cu")
+		(net "SUM")
+	)
+	(segment
+		(start 110.5375 108.675)
+		(end 111.75 108.675)
+		(width 0.2)
+		(layer "F.Cu")
+		(net "SUM")
+	)
+	(segment
+		(start 108.1 109)
+		(end 110.5375 108.675)
+		(width 0.2)
+		(layer "F.Cu")
+		(net "SUM")
+	)
+	(segment
+		(start 108.1 111.55)
+		(end 108.2 112.4)
+		(width 0.2)
+		(layer "F.Cu")
+		(net "SUM")
+	)
+	(segment
+		(start 106.15 112.05)
+		(end 106.15 113)
+		(width 0.2)
+		(layer "F.Cu")
+		(net "SUM")
+	)
+	(segment
+		(start 108.1 111.55)
+		(end 106.65 111.55)
+		(width 0.2)
+		(layer "F.Cu")
+		(net "SUM")
+	)
+	(segment
+		(start 111.75 108.675)
+		(end 111.75 111.525)
+		(width 0.2)
+		(layer "F.Cu")
+		(net "SUM")
+	)
+	(segment
+		(start 111.75 106.775)
+		(end 111.1875 105.9)
+		(width 0.2)
+		(layer "F.Cu")
+		(net "SUM")
+	)
+	(segment
+		(start 111.75 108.675)
+		(end 111.75 106.775)
+		(width 0.2)
+		(layer "F.Cu")
+		(net "SUM")
+	)
+	(segment
+		(start 108.1 109)
+		(end 108.1 111.55)
+		(width 0.2)
+		(layer "F.Cu")
+		(net "SUM")
+	)
+	(segment
+		(start 113.55 109.325)
+		(end 113.55 111.525)
+		(width 0.2)
+		(layer "F.Cu")
+		(net "TIA_OUT")
+	)
+	(segment
+		(start 113.55 106.775)
+		(end 114.1125 105.9)
+		(width 0.2)
+		(layer "F.Cu")
+		(net "TIA_OUT")
+	)
+	(segment
+		(start 115.9 109.325)
+		(end 115.9 110.55)
+		(width 0.2)
+		(layer "F.Cu")
+		(net "TIA_OUT")
+	)
+	(segment
+		(start 117.5 110.55)
+		(end 119 112.5)
+		(width 0.2)
+		(layer "F.Cu")
+		(net "TIA_OUT")
+	)
+	(segment
+		(start 117.975 109.875)
+		(end 118.5375 109)
+		(width 0.2)
+		(layer "F.Cu")
+		(net "TIA_OUT")
+	)
+	(segment
+		(start 113.55 109.325)
+		(end 113.55 106.775)
+		(width 0.2)
+		(layer "F.Cu")
+		(net "TIA_OUT")
+	)
+	(segment
+		(start 115.9 110.55)
+		(end 117.5 110.55)
+		(width 0.2)
+		(layer "F.Cu")
+		(net "TIA_OUT")
+	)
+	(segment
+		(start 113.55 111.525)
+		(end 113.425 112)
+		(width 0.2)
+		(layer "F.Cu")
+		(net "TIA_OUT")
+	)
+	(segment
+		(start 114.7625 109.325)
+		(end 115.9 109.325)
+		(width 0.2)
+		(layer "F.Cu")
+		(net "TIA_OUT")
+	)
+	(segment
+		(start 117.5 110.55)
+		(end 117.975 109.875)
+		(width 0.2)
+		(layer "F.Cu")
+		(net "TIA_OUT")
+	)
+	(segment
+		(start 114.7625 109.325)
+		(end 113.55 109.325)
+		(width 0.2)
+		(layer "F.Cu")
+		(net "TIA_OUT")
+	)
+	(segment
+		(start 114.7625 108.675)
+		(end 115.8 108.675)
+		(width 0.25)
+		(layer "F.Cu")
+		(net "AVDD_3V3")
+	)
+	(segment
+		(start 116.55 107.925)
+		(end 116.8 107.925)
+		(width 0.25)
+		(layer "F.Cu")
+		(net "AVDD_3V3")
+	)
+	(segment
+		(start 115.8 108.675)
+		(end 116.55 107.925)
+		(width 0.25)
+		(layer "F.Cu")
+		(net "AVDD_3V3")
 	)
 	(embedded_fonts no)

Commit message: Complete v0.4 final PCB routing
Routing:
- net AVDD_3V3: track 2.35 -> 92.1 mm
- net +5V_IN: track 0.00 -> 52.2 mm
- net CAL_IN: track 0.00 -> 34.3 mm
- net CAL_R_NODE: track 0.00 -> 29.7 mm
- net ADC_OUT: track 0.00 -> 27.1 mm
- net VREF_RAW: track 0.00 -> 23.0 mm
- net +5V_FILTER: track 0.00 -> 22.0 mm
- net AGND: track 1.23 -> 19.3 mm, vias 2 -> 18
- net VBIAS_1V25: track 0.00 -> 14.2 mm
- added copper zone on B.Cu, net AGND
Other:
- board text added: "OPEN"
- board text added: "SJCAL"
- board text added: "SUM_HIZ"
- board text added: "TP_CAL"
